File: PCB/iCE40_Breakout/power.kicad_sch (KiCad schematic)
At the start: 17 parts, among them U2 MIC5504-1.2YM5, U3 MIC5504-3.3YM5, U4 MIC5504-3.3YM5, U5 MIC5504-2.5YM5

Commit message: Changed all manually placed components into DNP, and changed the manually added caps to 0603
Parts:
- U2, U3, U4, U5: now not fitted
Changed lines of the file:
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@@
 		(in_bom yes)
 		(on_board yes)
-		(dnp no)
+		(dnp yes)
 		(fields_autoplaced yes)
 		(property "Reference" "U5"
@@
 		(in_bom yes)
 		(on_board yes)
-		(dnp no)
+		(dnp yes)
 		(fields_autoplaced yes)
 		(property "Reference" "U2"
@@
 		(in_bom yes)
 		(on_board yes)
-		(dnp no)
+		(dnp yes)
 		(fields_autoplaced yes)
 		(property "Reference" "U4"
@@
 		(in_bom yes)
 		(on_board yes)
-		(dnp no)
+		(dnp yes)
 		(fields_autoplaced yes)
 		(property "Reference" "U3"
